Commit message: Added collision, mass and inertia to the URDF. Work in progress on controllers and sensor plugins.

File: robot_design/urdf/robot_design.urdf (robot description, URDF)
Before this commit: robot autonomous_robot, 2 links, 1 joints
Links:
- link base_link: geometry collision box size=${base_length} ${base_width} ${base_height}; visual box size=${base_length} ${base_width} ${base_height}
Joints:
- joint base_joint: origin xyz=0.0 0.0 ${-(wheel_radius+wheel_zoff)} rpy=0 0 0 -> xyz=0.0 0.0 ${-(wheel_radius+wheel_back_zoff)} rpy=0 0 0

Commit message: Fixed link/joint issues, added counterweight to help with destabilisation when picking weights. Corrected some dimensioning issues. Working on the controllers and manipulator arm now!

File: robot_design/urdf/robot_design.urdf (robot description, URDF)
Before this commit: robot autonomous_robot, 2 links, 1 joints
Links:
- added link base_counterweight_link; collision box size=${base_length/2} ${base_width} ${base_height*2}; visual box size=${base_length/2} ${base_width} ${base_height*2}
Joints:
- added joint counter_weight_joint: type fixed, parent base_link, child base_counterweight_link, origin xyz=-0.315 0.0 0.090 rpy=0 0 0

Commit message: Added the manipulator arm necessary to pick up the boxes to the URDF. Collision, inertia and mass properties for the manipulator still in progress. The claw design can be improved.

File: robot_design/urdf/robot_design.urdf (robot description, URDF)
Before this commit: robot autonomous_robot, 3 links, 2 joints
Links:
- added link first_joint; visual cylinder length=0.4 radius=${cylinder_radius}
- added link first_joint_enclosure; visual box size=${base_length/5} ${base_width/5} ${base_height/2}
- added link grabber_fixture; visual box size=${base_length} ${base_width/5} ${base_height/3}
- added link grabber_fixture_left; visual cylinder length=0.3 radius=${cylinder_radius}
- added link grabber_fixture_right; visual cylinder length=0.3 radius=${cylinder_radius}
- added link left_gripper; visual mesh filename=package://urdf_tutorial/meshes/l_finger.dae
- added link left_tip; visual mesh filename=package://urdf_tutorial/meshes/l_finger_tip.dae
- added link right_gripper; visual mesh filename=package://urdf_tutorial/meshes/l_finger.dae
- added link right_tip; visual mesh filename=package://urdf_tutorial/meshes/l_finger_tip.dae
- added link second_joint; visual cylinder length=0.6 radius=${cylinder_radius}
- added link second_joint_enclosure; visual box size=${base_length/5} ${base_width/5} ${base_height/2}
- added link third_joint; visual cylinder length=0.2 radius=${cylinder_radius}
- added link third_joint_enclosure; visual box size=${base_length/5} ${base_width/5} ${base_height/2}
Joints:
- added joint first_joint_base: type revolute, parent base_link, child first_joint, origin xyz=0 0 0.09 rpy=0 1.5708 0, axis 0 1 0, limit lower=-0.7 upper=1.35 effort=1000.0 velocity=0.5
- added joint first_joint_enclosure_joint: type fixed, parent base_link, child first_joint_enclosure, origin xyz=0 0 0.13 rpy=0 0 0
- added joint grabber_fixture_joint: type fixed, parent third_joint, child grabber_fixture, origin xyz=0.2 0 0 rpy=0 0 0
- added joint grabber_fixture_left_joint: type prismatic, parent grabber_fixture, child grabber_fixture_left, origin xyz=0 0 0 rpy=0 0 0, axis 0 1 0, limit lower=0 upper=0.20 effort=1000.0 velocity=0.5
- added joint grabber_fixture_right_joint: type prismatic, parent grabber_fixture, child grabber_fixture_right, origin xyz=0 0 0 rpy=0 0 0, axis 0 -1 0, limit lower=0 upper=0.20 effort=1000.0 velocity=0.5
- added joint left_gripper_joint: type revolute, parent grabber_fixture_left, child left_gripper, origin xyz=0.02 0.28 0 rpy=0 0 0, axis 0 0 1, limit lower=-0.548 upper=0.548 effort=1000.0 velocity=0.5
- added joint left_tip_joint: type fixed, parent left_gripper, child left_tip
- added joint right_gripper_joint: type revolute, parent grabber_fixture_right, child right_gripper, origin xyz=0.02 -0.28 0 rpy=0 0 0, axis 0 0 -1, limit lower=-0.548 upper=0.548 effort=1000.0 velocity=0.5
- added joint right_tip_joint: type fixed, parent right_gripper, child right_tip
- added joint second_joint_base: type revolute, parent first_joint, child second_joint, origin xyz=-0.4 0 0 rpy=0 -1.5708 0, axis 0 1 0, limit lower=-1.0 upper=1.0 effort=1000.0 velocity=0.5
- added joint second_joint_enclosure_joint: type fixed, parent first_joint, child second_joint_enclosure, origin xyz=-0.4 0 0 rpy=0 0 0
- added joint third_joint_base: type revolute, parent second_joint, child third_joint, origin xyz=0.58 0 0 rpy=0 0 0, axis 0 1 0, limit lower=-1.35 upper=1.35 effort=1000.0 velocity=0.5
- added joint third_joint_enclosure_joint: type fixed, parent second_joint, child third_joint_enclosure, origin xyz=0.58 0 0 rpy=0 0 0

Commit message: Fixed wheels x position, fixed some inertia issues, mildly changed the visual design.

File: robot_design/urdf/robot_design.urdf (robot description, URDF)
Before this commit: robot autonomous_robot, 16 links, 15 joints
Links:
- removed link base_counterweight_link
- link first_joint_enclosure: geometry visual box size=${base_length/8} ${base_width/8} ${base_height/2}
- link grabber_fixture: geometry visual box size=${base_length/1.8} ${base_width/8} ${base_height/3}
- link second_joint_enclosure: geometry visual box size=${base_length/10} ${base_width/7} ${base_height/2}
- link third_joint_enclosure: geometry visual box size=${base_length/6} ${base_width/6} ${base_height/2}
Joints:
- removed joint counter_weight_joint

Commit message: Added colour and control plugins to the URDF for Gazebo.

File: robot_design/urdf/robot_design.urdf (robot description, URDF)
Before this commit: robot autonomous_robot, 15 links, 14 joints
Links:
- link first_joint: geometry collision cylinder length=${0.4/scale} radius=${cylinder_radius}; visual cylinder length=${0.4/scale} radius=${cylinder_radius}
- link first_joint_enclosure: geometry collision box size=${base_length/8} ${base_width/8} ${base_height/2}; visual box size=${base_length/8} ${base_width/8} ${base_height/2}
- link grabber_fixture: geometry collision box size=${base_length/1.8} ${base_width/8} ${base_height/3}; visual box size=${base_length/1.8} ${base_width/8} ${base_height/3}
- link grabber_fixture_left: geometry visual cylinder length=${0.3/scale} radius=${cylinder_radius}
- link grabber_fixture_right: geometry visual cylinder length=${0.3/scale} radius=${cylinder_radius}
- link second_joint: geometry collision cylinder length=${0.6/scale} radius=${cylinder_radius}; visual cylinder length=${0.6/scale} radius=${cylinder_radius}
- link second_joint_enclosure: geometry collision box size=${base_length/10} ${base_width/7} ${base_height/2}; visual box size=${base_length/10} ${base_width/7} ${base_height/2}
- link third_joint: geometry collision cylinder length=${0.2/scale} radius=${cylinder_radius}; visual cylinder length=${0.2/scale} radius=${cylinder_radius}
- link third_joint_enclosure: geometry collision box size=${base_length/6} ${base_width/6} ${base_height/2}; visual box size=${base_length/6} ${base_width/6} ${base_height/2}

Commit message: Fixed sliding errors by changing inertia. Added hardware interface plugin for Gazebo to URDF. Added controllers. Added yaml file for the joint configurations. Added launch file. The robot can now be moved around using the URDF_Tutorial DIFF Driver Controller GUI or with teleop.

File: robot_design/urdf/robot_design.urdf (robot description, URDF)
Before this commit: robot autonomous_robot, 15 links, 14 joints
Links:
- link grabber_fixture_left: geometry collision cylinder length=${0.3/scale} radius=${cylinder_radius}; visual cylinder length=${0.3/scale} radius=${cylinder_radius}
- link grabber_fixture_right: geometry collision cylinder length=${0.3/scale} radius=${cylinder_radius}; visual cylinder length=${0.3/scale} radius=${cylinder_radius}
- link left_gripper: geometry collision mesh filename=package://urdf_tutorial/meshes/l_finger.dae; visual mesh filename=package://urdf_tutorial/meshes/l_finger.dae
- link left_tip: geometry collision mesh filename=package://urdf_tutorial/meshes/l_finger_tip.dae; visual mesh filename=package://urdf_tutorial/meshes/l_finger_tip.dae
- link right_gripper: geometry collision mesh filename=package://urdf_tutorial/meshes/l_finger.dae; visual mesh filename=package://urdf_tutorial/meshes/l_finger.dae
- link right_tip: geometry collision mesh filename=package://urdf_tutorial/meshes/l_finger_tip.dae; visual mesh filename=package://urdf_tutorial/meshes/l_finger_tip.dae

Commit message: Full scalability added to the URDF file, now the robot can be used with any Gazebo Wolrd and with any dimensioning. Fixed Tiff error in RVIZ from loading DAE files (bug present on Noetic + Gazebo v9 and over). Removed dependency on URDF_Tutorial package by creating a meshes folder available within the robot_design package itself.

File: robot_design/urdf/robot_design.urdf (robot description, URDF)
Before this commit: robot autonomous_robot, 15 links, 14 joints
Links:
- added link dummy
- link left_gripper: geometry collision mesh filename=package://robot_design/meshes/l_finger.dae scale=${1/scale} ${1/scale} ${1/scale}; visual mesh filename=package://robot_design/meshes/l_finger.dae scale=${1/scale} ${1/scale} ${1/scale}
- link left_tip: geometry collision mesh filename=package://robot_design/meshes/l_finger_tip.dae scale=${1/scale} ${1/scale} ${1/scale}; visual mesh filename=package://robot_design/meshes/l_finger_tip.dae scale=${1/scale} ${1/scale} ${1/scale}
- link right_gripper: geometry collision mesh filename=package://robot_design/meshes/l_finger.dae scale=${1/scale} ${1/scale} ${1/scale}; visual mesh filename=package://robot_design/meshes/l_finger.dae scale=${1/scale} ${1/scale} ${1/scale}
- link right_tip: geometry collision mesh filename=package://robot_design/meshes/l_finger_tip.dae scale=${1/scale} ${1/scale} ${1/scale}; visual mesh filename=package://robot_design/meshes/l_finger_tip.dae scale=${1/scale} ${1/scale} ${1/scale}
Joints:
- added joint dummy_joint: type fixed, parent dummy, child base_link
- joint base_joint: origin xyz=0.0 0.0 ${-(wheel_radius+wheel_back_zoff)} rpy=0 0 0 -> xyz=${0.0/scale} ${0.0/scale} ${-(wheel_radius+wheel_back_zoff)} rpy=0 0 0
- joint first_joint_base: origin xyz=0 0 0.09 rpy=0 1.5708 0 -> xyz=${0/scale} ${0/scale} ${0.09/scale} rpy=0 1.5708 0
- joint first_joint_enclosure_joint: origin xyz=0 0 0.13 rpy=0 0 0 -> xyz=${0/scale} ${0/scale} ${0.13/scale} rpy=0 0 0
- joint grabber_fixture_joint: origin xyz=0.2 0 0 rpy=0 0 0 -> xyz=${0.2/scale} ${0/scale} ${0/scale} rpy=0 0 0
- joint grabber_fixture_left_joint: origin xyz=0 0 0 rpy=0 0 0 -> xyz=${0/scale} ${0/scale} ${0/scale} rpy=0 0 0
- joint grabber_fixture_right_joint: origin xyz=0 0 0 rpy=0 0 0 -> xyz=${0/scale} ${0/scale} ${0/scale} rpy=0 0 0
- joint left_gripper_joint: origin xyz=0.02 0.28 0 rpy=0 0 0 -> xyz=${0.02/scale} ${0.28/scale} ${0/scale} rpy=0 0 0
- joint right_gripper_joint: origin xyz=0.02 -0.28 0 rpy=0 0 0 -> xyz=${0.02/scale} ${-0.28/scale} ${0/scale} rpy=0 0 0
- joint second_joint_base: origin xyz=-0.4 0 0 rpy=0 -1.5708 0 -> xyz=${-0.4/scale} ${0/scale} ${0/scale} rpy=0 -1.5708 0
- joint second_joint_enclosure_joint: origin xyz=-0.4 0 0 rpy=0 0 0 -> xyz=${-0.4/scale} ${0/scale} ${0/scale} rpy=0 0 0
- joint third_joint_base: origin xyz=0.58 0 0 rpy=0 0 0 -> xyz=${0.58/scale} ${0/scale} ${0/scale} rpy=0 0 0
- joint third_joint_enclosure_joint: origin xyz=0.58 0 0 rpy=0 0 0 -> xyz=${0.58/scale} ${0/scale} ${0/scale} rpy=0 0 0

Commit message: Moved the manipulator arm to the front of the chassis. Added a laser scanner on top of the chassis in the center. Added gazebo plugins for odometry and laser scan topics. Launch files updated to include RVIZ, the robot is now fully functional. Added an extra instructions file with different robot launch states.

File: robot_design/urdf/robot_design.urdf (robot description, URDF)
Before this commit: robot autonomous_robot, 16 links, 15 joints
Links:
- added link sensor_laser; collision cylinder length=${0.06/scale} radius=${cylinder_radius*5}; visual cylinder length=${0.06/scale} radius=${cylinder_radius*5}
- link left_gripper: geometry collision mesh filename=package://robot_design/meshes/l_finger.dae scale=${0.5/scale} ${0.5/scale} ${0.5/scale}; visual mesh filename=package://robot_design/meshes/l_finger.dae scale=${0.5/scale} ${0.5/scale} ${0.5/scale}
- link left_tip: geometry collision mesh filename=package://robot_design/meshes/l_finger_tip.dae scale=${0.5/scale} ${0.5/scale} ${0.5/scale}; visual mesh filename=package://robot_design/meshes/l_finger_tip.dae scale=${0.5/scale} ${0.5/scale} ${0.5/scale}
- link right_gripper: geometry collision mesh filename=package://robot_design/meshes/l_finger.dae scale=${0.5/scale} ${0.5/scale} ${0.5/scale}; visual mesh filename=package://robot_design/meshes/l_finger.dae scale=${0.5/scale} ${0.5/scale} ${0.5/scale}
- link right_tip: geometry collision mesh filename=package://robot_design/meshes/l_finger_tip.dae scale=${0.5/scale} ${0.5/scale} ${0.5/scale}; visual mesh filename=package://robot_design/meshes/l_finger_tip.dae scale=${0.5/scale} ${0.5/scale} ${0.5/scale}
Joints:
- added joint joint_sensor_laser: type fixed, parent base_link, child sensor_laser, origin xyz=${0/scale} ${0/scale} ${0.12/scale} rpy=0 0 0
- joint first_joint_base: origin xyz=${0/scale} ${0/scale} ${0.09/scale} rpy=0 1.5708 0 -> xyz=${0.30/scale} ${0/scale} ${0.09/scale} rpy=0 1.5708 0
- joint first_joint_enclosure_joint: origin xyz=${0/scale} ${0/scale} ${0.13/scale} rpy=0 0 0 -> xyz=${0.30/scale} ${0/scale} ${0.13/scale} rpy=0 0 0

Commit message: Added costmap local/global and base banner parameters yaml files for the Navigation Stack. Added IMU to the URDF.

File: robot_design/urdf/robot_design.urdf (robot description, URDF)
Before this commit: robot autonomous_robot, 17 links, 16 joints
Links:
- added link imu_link, mass ${0.001/scale}; collision box size=.001 .001 .001; visual box size=0.001 0.001 0.001
Joints:
- added joint imu_joint: type fixed, parent base_link, child imu_link, origin xyz=-0.350 0 0.115, axis 1 0 0

Commit message: Worked on the controller and the RVIZ tree. Some issues with the transfer frames. Navigation stack still WIP!

File: robot_design/urdf/robot_design.urdf (robot description, URDF)
Before this commit: robot autonomous_robot, 18 links, 17 joints
Links:
- removed link dummy
- removed link imu_link
- added link sensor_imu, mass ${0.001/scale}; collision box size=.001 .001 .001; visual box size=0.001 0.001 0.001
Joints:
- removed joint dummy_joint
- joint base_joint: origin xyz=${0.0/scale} ${0.0/scale} ${-(wheel_radius+wheel_back_zoff)} rpy=0 0 0 -> xyz=0.0 0.0 ${-(wheel_radius+wheel_back_zoff)} rpy=0 0 0
- joint imu_joint: child imu_link -> sensor_imu

Commit message: Moved the robot arm backwards to reduce robot footprint. Fixed IMU sensor location.

File: robot_design/urdf/robot_design.urdf (robot description, URDF)
Before this commit: robot autonomous_robot, 16 links, 15 joints
Links:
- link sensor_imu: geometry collision box size=${base_length/10} ${base_width/10} ${base_height/10}; visual box size=${base_length/10} ${base_width/10} ${base_height/10}
Joints:
- joint imu_joint: origin xyz=-0.350 0 0.115 -> xyz=${0/scale} ${0/scale} ${-0.05/scale}
- joint second_joint_base: limit lower=-1.0 upper=1.0 effort=1000.0 velocity=0.5 -> lower=0.0 upper=4.2 effort=1000.0 velocity=0.5; origin xyz=${-0.4/scale} ${0/scale} ${0/scale} rpy=0 -1.5708 0 -> xyz=${-0.4/scale} ${0/scale} ${0/scale} rpy=0 1.5708 0
- joint third_joint_base: origin xyz=${0.58/scale} ${0/scale} ${0/scale} rpy=0 0 0 -> xyz=${0.58/scale} ${0/scale} ${0/scale} rpy=0 -1.5708 0

Commit message: Some more progress on the navigation, but it is still not functional.

File: robot_design/urdf/robot_design.urdf (robot description, URDF)
Before this commit: robot autonomous_robot, 16 links, 15 joints
Joints:
- joint first_joint_base: origin xyz=${0.30/scale} ${0/scale} ${0.09/scale} rpy=0 1.5708 0 -> xyz=${-0.30/scale} ${0/scale} ${0.09/scale} rpy=0 1.5708 0
- joint first_joint_enclosure_joint: origin xyz=${0.30/scale} ${0/scale} ${0.13/scale} rpy=0 0 0 -> xyz=${-0.30/scale} ${0/scale} ${0.13/scale} rpy=0 0 0
- joint second_joint_base: origin xyz=${-0.4/scale} ${0/scale} ${0/scale} rpy=0 1.5708 0 -> xyz=${-0.4/scale} ${0/scale} ${0/scale} rpy=0 -1.5708 0
- joint third_joint_base: origin xyz=${0.58/scale} ${0/scale} ${0/scale} rpy=0 -1.5708 0 -> xyz=${0.58/scale} ${0/scale} ${0/scale} rpy=0 1.5708 0

Commit message: Fixed inertia values/functions for URDF. Fixed some scalling issues. Changed costmaps, changed launchfiles regarding move base and AMCL. Changed RVIZ configuration file.

File: robot_design/urdf/robot_design.urdf (robot description, URDF)
Before this commit: robot autonomous_robot, 16 links, 15 joints
Links:
- link left_gripper: geometry collision mesh filename=package://robot_design/meshes/l_finger.dae scale=${1/scale} ${1/scale} ${1/scale}; visual mesh filename=package://robot_design/meshes/l_finger.dae scale=${1/scale} ${1/scale} ${1/scale}
- link left_tip: geometry collision mesh filename=package://robot_design/meshes/l_finger_tip.dae scale=${1/scale} ${1/scale} ${1/scale}; visual mesh filename=package://robot_design/meshes/l_finger_tip.dae scale=${1/scale} ${1/scale} ${1/scale}
- link right_gripper: geometry collision mesh filename=package://robot_design/meshes/l_finger.dae scale=${1/scale} ${1/scale} ${1/scale}; visual mesh filename=package://robot_design/meshes/l_finger.dae scale=${1/scale} ${1/scale} ${1/scale}
- link right_tip: geometry collision mesh filename=package://robot_design/meshes/l_finger_tip.dae scale=${1/scale} ${1/scale} ${1/scale}; visual mesh filename=package://robot_design/meshes/l_finger_tip.dae scale=${1/scale} ${1/scale} ${1/scale}
Joints:
- joint imu_joint: origin xyz=${0/scale} ${0/scale} ${-0.05/scale} -> xyz=${0/scale} ${0/scale} ${-0.1/scale}
