Commit message: Changed directory structure to be more organised. Moved the robot URDF inside the package so only 1 package required. Edited the cost maps. Changed from P3D Odometry solution to Diff_drive_controller odometry solution which was already implemented. Reduced robot size by 17% with the scale function. Added extra comments to launch files and URDF. Navigation stack is now almost fully working. Issue with laser position/odometry value. To be fixed.

File: models/robot_design/urdf/robot_design.urdf (robot description, URDF)
Before this commit: robot autonomous_robot, 16 links, 15 joints
Links:
- added link chassis; collision box size=${base_length} ${base_width} ${base_height}; visual box size=${base_length} ${base_width} ${base_height}
- link base_link: geometry 
- link left_gripper: geometry collision mesh filename=package://assessmentmobilerobots_2022/models/robot_design/m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 scale=${1/scale} ${1/scale} ${1/scale}; visual mesh filename=package://assessmentmobilerobots_2022/models/robot_design/m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 scale=${1/scale} ${1/scale} ${1/scale}
- link left_tip: geometry collision mesh filename=package://assessmentmobilerobots_2022/models/robot_design/m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 scale=${1/scale} ${1/scale} ${1/scale}; visual mesh filename=package://assessmentmobilerobots_2022/models/robot_design/m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 scale=${1/scale} ${1/scale} ${1/scale}
- link right_gripper: geometry collision mesh filename=package://assessmentmobilerobots_2022/models/robot_design/m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 scale=${1/scale} ${1/scale} ${1/scale}; visual mesh filename=package://assessmentmobilerobots_2022/models/robot_design/m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 scale=${1/scale} ${1/scale} ${1/scale}
- link right_tip: geometry collision mesh filename=package://assessmentmobilerobots_2022/models/robot_design/m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 scale=${1/scale} ${1/scale} ${1/scale}; visual mesh filename=package://assessmentmobilerobots_2022/models/robot_design/m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 scale=${1/scale} ${1/scale} ${1/scale}
Joints:
- added joint base_link_joint: type fixed, parent base_link, child chassis
- joint first_joint_base: parent base_link -> chassis
- joint first_joint_enclosure_joint: parent base_link -> chassis
- joint imu_joint: parent base_link -> chassis
- joint joint_sensor_laser: parent base_link -> chassis

Commit message: Fixed the PID controller for all joints. Added an initial pose for the whole manipulator arm in the launch file. Added a camera for Computer Vision, to be used to detect boxes and their height from the ground. Dedicated about a dozen hours to optimising the odometry values with not much luck, forward/backwards movement is now highly accurate, but rotation is still not great, although better than before.

File: models/robot_design/urdf/robot_design.urdf (robot description, URDF)
Before this commit: robot autonomous_robot, 17 links, 16 joints
Links:
- added link camera; collision box size=${camera_size} ${camera_size} ${camera_size}; visual box size=${camera_size} ${camera_size} ${camera_size}
Joints:
- added joint camera_joint: type fixed, parent chassis, child camera, origin xyz=0.155 0 0 rpy=0 0 0

Commit message: Better formatted the URDF and added extra comments. Added an extra prismatic joint, modified the ranges of some other joints. Added RVIZ Visualization and joint control launch file and configuration.

File: models/robot_design/urdf/robot_design.urdf (robot description, URDF)
Before this commit: robot autonomous_robot, 18 links, 17 joints
Links:
- link second_joint_enclosure: geometry collision box size=${base_length/10} ${base_width/7} ${base_height*4}; visual box size=${base_length/10} ${base_width/7} ${base_height*4}
Joints:
- joint second_joint_base: axis 0 1 0 -> 1 0 0; limit lower=0.0 upper=4.2 effort=1000.0 velocity=0.5 -> lower=0 upper=0.15 effort=1000.0 velocity=0.5; origin xyz=${-0.4/scale} ${0/scale} ${0/scale} rpy=0 -1.5708 0 -> xyz=${0.0/scale} ${0/scale} ${-0.10/scale} rpy=0 -1.5708 0; parent first_joint -> second_joint_enclosure; type revolute -> prismatic
- joint second_joint_enclosure_joint: axis (none) -> 0 1 0; limit (none) -> lower=-0.15 upper=0.15 effort=1000.0 velocity=0.5; origin xyz=${-0.4/scale} ${0/scale} ${0/scale} rpy=0 0 0 -> xyz=${-0.4/scale} ${0/scale} ${0.3/scale} rpy=0 0 0; type fixed -> revolute
- joint third_joint_base: limit lower=-1.35 upper=1.35 effort=1000.0 velocity=0.5 -> lower=-2.5 upper=1.00 effort=1000.0 velocity=0.5

Commit message: Reduced joints force/effort, increased velocity, in URDF. Added joint publisher python script and found default positions to be executed.

File: models/robot_design/urdf/robot_design.urdf (robot description, URDF)
Before this commit: robot autonomous_robot, 18 links, 17 joints
Joints:
- joint first_joint_base: limit lower=-0.7 upper=1.35 effort=1000.0 velocity=0.5 -> lower=-0.7 upper=1.35 effort=5.0 velocity=5.0
- joint grabber_fixture_left_joint: limit lower=0 upper=0.20 effort=1000.0 velocity=0.5 -> lower=0 upper=0.20 effort=5.0 velocity=5.0
- joint grabber_fixture_right_joint: limit lower=0 upper=0.20 effort=1000.0 velocity=0.5 -> lower=0 upper=0.20 effort=5.0 velocity=5.0
- joint left_gripper_joint: limit lower=-0.548 upper=0.548 effort=1000.0 velocity=0.5 -> lower=-0.548 upper=0.548 effort=5.0 velocity=5.0
- joint right_gripper_joint: limit lower=-0.548 upper=0.548 effort=1000.0 velocity=0.5 -> lower=-0.548 upper=0.548 effort=5.0 velocity=5.0
- joint second_joint_base: limit lower=0 upper=0.15 effort=1000.0 velocity=0.5 -> lower=0 upper=0.15 effort=5.0 velocity=5.0
- joint second_joint_enclosure_joint: limit lower=-0.15 upper=0.15 effort=1000.0 velocity=0.5 -> lower=-0.15 upper=0.15 effort=5.0 velocity=5.0
- joint third_joint_base: limit lower=-2.5 upper=1.00 effort=1000.0 velocity=0.5 -> lower=-2.5 upper=1.00 effort=5.0 velocity=5.0

Commit message: Added prismatic joint scaling to the scalling factor. Reduced size of claw to better grasp cubes. Added Gazebo Grasping Tag/Hack.

File: models/robot_design/urdf/robot_design.urdf (robot description, URDF)
Before this commit: robot autonomous_robot, 18 links, 17 joints
Links:
- link grabber_fixture: geometry collision box size=${base_length/3.5} ${base_width/8} ${base_height/3}; visual box size=${base_length/3.5} ${base_width/8} ${base_height/3}
- link grabber_fixture_left: geometry collision cylinder length=${0.15/scale} radius=${cylinder_radius}; visual cylinder length=${0.15/scale} radius=${cylinder_radius}
- link grabber_fixture_right: geometry collision cylinder length=${0.15/scale} radius=${cylinder_radius}; visual cylinder length=${0.15/scale} radius=${cylinder_radius}
Joints:
- joint grabber_fixture_left_joint: limit lower=0 upper=0.20 effort=5.0 velocity=5.0 -> lower=${-0.18/(scale*scale)} upper=${0.18/(scale*scale)} effort=5.0 velocity=5.0
- joint grabber_fixture_right_joint: limit lower=0 upper=0.20 effort=5.0 velocity=5.0 -> lower=${-0.18/(scale*scale)} upper=${0.18/(scale*scale)} effort=5.0 velocity=5.0
- joint left_gripper_joint: origin xyz=${0.02/scale} ${0.28/scale} ${0/scale} rpy=0 0 0 -> xyz=${0.02/scale} ${0.20/scale} ${0/scale} rpy=0 0 0
- joint right_gripper_joint: origin xyz=${0.02/scale} ${-0.28/scale} ${0/scale} rpy=0 0 0 -> xyz=${0.02/scale} ${-0.20/scale} ${0/scale} rpy=0 0 0
- joint second_joint_base: limit lower=0 upper=0.15 effort=5.0 velocity=5.0 -> lower=0 upper=${1.3/(scale*scale)} effort=5.0 velocity=5.0

Commit message: Fixed move_boxes script that had an error if the controllers had a delay in loading (example high cpu usage). Modified claw again, made it smalled, made prismatic joint longer. OPtimised Gazebo Grasp tag/hack to require less time, 20seconds is the best achieved.

File: models/robot_design/urdf/robot_design.urdf (robot description, URDF)
Before this commit: robot autonomous_robot, 18 links, 17 joints
Links:
- link grabber_fixture: geometry collision box size=${base_length/5.0} ${base_width/8} ${base_height/3}; visual box size=${base_length/5.0} ${base_width/8} ${base_height/3}
- link grabber_fixture_left: geometry collision cylinder length=${0.12/scale} radius=${cylinder_radius}; visual cylinder length=${0.08/scale} radius=${cylinder_radius}
- link grabber_fixture_right: geometry collision cylinder length=${0.15/scale} radius=${cylinder_radius}; visual cylinder length=${0.08/scale} radius=${cylinder_radius}
- link second_joint: geometry collision cylinder length=${0.6/scale} radius=${cylinder_radius}; visual cylinder length=${0.9/scale} radius=${cylinder_radius}
Joints:
- joint grabber_fixture_left_joint: limit lower=${-0.18/(scale*scale)} upper=${0.18/(scale*scale)} effort=5.0 velocity=5.0 -> lower=${-0.24/(scale*scale)} upper=${0.1/(scale*scale)} effort=5.0 velocity=5.0
- joint grabber_fixture_right_joint: limit lower=${-0.18/(scale*scale)} upper=${0.18/(scale*scale)} effort=5.0 velocity=5.0 -> lower=${-0.24/(scale*scale)} upper=${0.1/(scale*scale)} effort=5.0 velocity=5.0
- joint left_gripper_joint: origin xyz=${0.02/scale} ${0.20/scale} ${0/scale} rpy=0 0 0 -> xyz=${0.02/scale} ${0.18/scale} ${0/scale} rpy=0 0 0
- joint right_gripper_joint: origin xyz=${0.02/scale} ${-0.20/scale} ${0/scale} rpy=0 0 0 -> xyz=${0.02/scale} ${-0.18/scale} ${0/scale} rpy=0 0 0
- joint second_joint_base: limit lower=0 upper=${1.3/(scale*scale)} effort=5.0 velocity=5.0 -> lower=0.0 upper=${1.9/(scale*scale)} effort=5.0 velocity=5.0; origin xyz=${0.0/scale} ${0/scale} ${-0.10/scale} rpy=0 -1.5708 0 -> xyz=${0.0/scale} ${0/scale} ${-0.13/scale} rpy=0 -1.5708 0
- joint third_joint_base: origin xyz=${0.58/scale} ${0/scale} ${0/scale} rpy=0 1.5708 0 -> xyz=${0.7/scale} ${0/scale} ${0/scale} rpy=0 1.5708 0
- joint third_joint_enclosure_joint: origin xyz=${0.58/scale} ${0/scale} ${0/scale} rpy=0 0 0 -> xyz=${0.7/scale} ${0/scale} ${0/scale} rpy=0 0 0

Commit message: Changed package name. Updated Readme. Updated launch files to reflect the name change. Fixed some map issues.

File: models/robot_design/urdf/robot_design.urdf (robot description, URDF)
Before this commit: robot autonomous_robot, 18 links, 17 joints
Links:
- link left_gripper: geometry collision mesh filename=package://ros_autonomous_manipulator_mobilerobot/models/rob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 scale=${1/scale} ${1/scale} ${1/scale}; visual mesh filename=package://ros_autonomous_manipulator_mobilerobot/models/rob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 scale=${1/scale} ${1/scale} ${1/scale}
- link left_tip: geometry collision mesh filename=package://ros_autonomous_manipulator_mobilerobot/models/rob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 scale=${1/scale} ${1/scale} ${1/scale}; visual mesh filename=package://ros_autonomous_manipulator_mobilerobot/models/rob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 scale=${1/scale} ${1/scale} ${1/scale}
- link right_gripper: geometry collision mesh filename=package://ros_autonomous_manipulator_mobilerobot/models/rob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 scale=${1/scale} ${1/scale} ${1/scale}; visual mesh filename=package://ros_autonomous_manipulator_mobilerobot/models/rob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 scale=${1/scale} ${1/scale} ${1/scale}
- link right_tip: geometry collision mesh filename=package://ros_autonomous_manipulator_mobilerobot/models/rob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 scale=${1/scale} ${1/scale} ${1/scale}; visual mesh filename=package://ros_autonomous_manipulator_mobilerobot/models/rob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 scale=${1/scale} ${1/scale} ${1/scale}
